File: XiaoCarrierARGB.kicad_pcb (KiCad board)
At the start: 4 copper layers, 63.5 x 38.1 mm, 43 parts, among them J1 V_{IN}^{10-24V}, J2 Conn_01x08, J3 Conn_01x01, J4 Conn_01x08, J5 Conn_01x01, J6 Conn_01x06, U1 TLV75733PDBV, U2 TPP362083-T6TR, U3 XIAO-ESP32-C6-DIP, U4 74LVC1T45W6-7, U5 74LVC1T45W6-7, U6 74LVC1T45W6-7

Commit message: Finished up layout
Need to do final sanity checks BUCK and such
Parts:
- added C8: 100n, Capacitor_SMD:C_0805_2012Metric_Pad1.18x1.45mm_HandSolder, F.Cu at (96.7, 94.5)
- moved JP10 3.40 mm to (99.5, 91.0), turned to 90 degrees
- moved JP12 0.86 mm to (127.5, 94.0)
- moved C7 0.74 mm to (108.2, 94.2)
- moved C6 0.56 mm to (108.2, 90.3)
- moved R10 0.52 mm to (137.9, 86.5)
- moved R9 0.51 mm to (135.4, 86.5)
- moved C1 0.39 mm to (98.5, 111.0)
- moved U1 0.30 mm to (102.0, 110.9)
- moved R6 0.30 mm to (104.5, 86.5)
- moved JP9 0.20 mm to (117.0, 94.0)
- moved R5 0.16 mm to (107.1, 86.5)
- moved JP14 0.14 mm to (142.2, 90.9)
- moved C4 0.11 mm to (102.1, 114.3)
- moved R4 0.10 mm to (114.7, 86.5)
- turned JP11 to 0 degrees
Connections:
- R11 pad 1: /LED_DATA^{1} -> Net-(J6-Pin_1)
- R11 pad 2: Net-(J6-Pin_1) -> /LED_DATA^{1}
- R12 pad 1: /LED_DATA^{2} -> Net-(J6-Pin_3)
- R12 pad 2: Net-(J6-Pin_3) -> /LED_DATA^{2}
- R13 pad 1: /LED_DATA^{3} -> Net-(J6-Pin_5)
- R13 pad 2: Net-(J6-Pin_5) -> /LED_DATA^{3}
Routing:
- net +3V3: track 0.00 -> 153.7 mm, vias 0 -> 7
- net +5V: track 0.00 -> 103.4 mm, vias 0 -> 9
- net /Xiao3v3: track 0.00 -> 47.9 mm, vias 0 -> 3
- net GND: track 0.00 -> 36.8 mm, vias 0 -> 21
- net /GPIO2: track 0.00 -> 19.9 mm
- net /GPIO1: track 0.00 -> 17.1 mm
- net /GPIO0: track 0.00 -> 14.0 mm
- net Net-(JP13-C): track 0.00 -> 6.13 mm
- net Net-(JP11-C): track 0.00 -> 6.13 mm
- net Net-(JP8-C): track 0.00 -> 5.98 mm
- net Net-(JP15-C): track 0.00 -> 5.98 mm
- net Net-(JP14-C): track 0.00 -> 4.70 mm
- net Net-(J6-Pin_5): track 0.00 -> 4.68 mm
- net Net-(J6-Pin_3): track 0.00 -> 4.68 mm
- net Net-(J6-Pin_1): track 0.00 -> 4.68 mm
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- added copper zone on B.Cu, net +3V3
- added copper zone on F.Cu, net +3V3
- added copper zone on B.Cu, net +5V
- added copper zone on F.Cu, net +5V
- added copper zone on F.Cu, net /LDO_{in}
- added copper zone on F.Cu, net /SWITCHNODE
- added copper zone on F.Cu, net /V_{IN}
- added copper zone on F.Cu, net /V_{IN}_{FUSED}

Commit message: Added ground fills to top and bottom layers Silkscreen layout needs to be done for easy pin ID
Routing:
- net GND: vias 21 -> 45
- added copper zone on B.Cu, net GND
- added copper zone on F.Cu, net GND
Changed lines of the file:
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@@
+	)
+	(via
+		(at 120.85 98.85)
+		(size 0.6)
+		(drill 0.3)
+		(layers "F.Cu" "B.Cu")
+		(free yes)
+		(net "GND")
 	)
 	(via
@@
 		(drill 0.3)
 		(layers "F.Cu" "B.Cu")
+		(net "GND")
+	)
+	(via
+		(at 116.45 99.45)
+		(size 0.6)
+		(drill 0.3)
+		(layers "F.Cu" "B.Cu")
+		(free yes)
+		(net "GND")
+	)
+	(via
+		(at 120.85 102.85)
+		(size 0.6)
+		(drill 0.3)
+		(layers "F.Cu" "B.Cu")
+		(free yes)
 		(net "GND")
 	)
@@
 	)
 	(via
+		(at 116.65 106.65)
+		(size 0.6)
+		(drill 0.3)
+		(layers "F.Cu" "B.Cu")
+		(free yes)
+		(net "GND")
+	)
+	(via
+		(at 129.05 90.65)
+		(size 0.6)
+		(drill 0.3)
+		(layers "F.Cu" "B.Cu")
+		(free yes)
+		(net "GND")
+	)
+	(via
+		(at 116.65 109.05)
+		(size 0.6)
+		(drill 0.3)
+		(layers "F.Cu" "B.Cu")
+		(free yes)
+		(net "GND")
+	)
+	(via
 		(at 108.519962 95.162607)
 		(size 0.7)
@@
 	)
 	(via
+		(at 125.45 109.05)
+		(size 0.6)
+		(drill 0.3)
+		(layers "F.Cu" "B.Cu")
+		(free yes)
+		(net "GND")
+	)
+	(via
+		(at 120.85 109.05)
+		(size 0.6)
+		(drill 0.3)
+		(layers "F.Cu" "B.Cu")
+		(free yes)
+		(net "GND")
+	)
+	(via
+		(at 126.85 100.25)
+		(size 0.6)
+		(drill 0.3)
+		(layers "F.Cu" "B.Cu")
+		(free yes)
+		(net "GND")
+	)
+	(via
 		(at 109.35 88.95)
 		(size 0.7)
@@
 	)
 	(via
+		(at 127.25 95.85)
+		(size 0.6)
+		(drill 0.3)
+		(layers "F.Cu" "B.Cu")
+		(free yes)
+		(net "GND")
+	)
+	(via
 		(at 109.225 95.525)
 		(size 0.6)
@@
 	)
 	(via
+		(at 123.85 106.65)
+		(size 0.6)
+		(drill 0.3)
+		(layers "F.Cu" "B.Cu")
+		(free yes)
+		(net "GND")
+	)
+	(via
+		(at 118.45 106.65)
+		(size 0.6)
+		(drill 0.3)
+		(layers "F.Cu" "B.Cu")
+		(free yes)
+		(net "GND")
+	)
+	(via
 		(at 90.25 93.5)
 		(size 0.7)
@@
 	)
 	(via
+		(at 113.25 91.65)
+		(size 0.6)
+		(drill 0.3)
+		(layers "F.Cu" "B.Cu")
+		(free yes)
+		(net "GND")
+	)
+	(via
+		(at 115.05 109.05)
+		(size 0.6)
+		(drill 0.3)
+		(layers "F.Cu" "B.Cu")
+		(free yes)
+		(net "GND")
+	)
+	(via
+		(at 118.45 109.05)
+		(size 0.6)
+		(drill 0.3)
+		(layers "F.Cu" "B.Cu")
+		(free yes)
+		(net "GND")
+	)
+	(via
+		(at 133.25 86.65)
+		(size 0.6)
+		(drill 0.3)
+		(layers "F.Cu" "B.Cu")
+		(free yes)
+		(net "GND")
+	)
+	(via
 		(at 102 110.9)
 		(size 0.7)
@@
 	)
 	(via
+		(at 114.85 103.05)
+		(size 0.6)
+		(drill 0.3)
+		(layers "F.Cu" "B.Cu")
+		(free yes)
+		(net "GND")
+	)
+	(via
+		(at 123.85 109.05)
+		(size 0.6)
+		(drill 0.3)
+		(layers "F.Cu" "B.Cu")
+		(free yes)
+		(net "GND")
+	)
+	(via
+		(at 116.45 84.65)
+		(size 0.6)
+		(drill 0.3)
+		(layers "F.Cu" "B.Cu")
+		(free yes)
+		(net "GND")
+	)
+	(via
 		(at 133.45 90.85)
 		(size 0.7)
@@
 	)
 	(via
+		(at 120.85 106.65)
+		(size 0.6)
+		(drill 0.3)
+		(layers "F.Cu" "B.Cu")
+		(free yes)
+		(net "GND")
+	)
+	(via
+		(at 113.25 95.05)
+		(size 0.6)
+		(drill 0.3)
+		(layers "F.Cu" "B.Cu")
+		(free yes)
+		(net "GND")
+	)
+	(via
+		(at 118.45 98.85)
+		(size 0.6)
+		(drill 0.3)
+		(layers "F.Cu" "B.Cu")
+		(free yes)
+		(net "GND")
+	)
+	(via
+		(at 118.45 102.85)
+		(size 0.6)
+		(drill 0.3)
+		(layers "F.Cu" "B.Cu")
+		(free yes)
+		(net "GND")
+	)
+	(via
 		(at 108.9 99.1)
 		(size 0.6)
@@
 		(drill 0.3)
 		(layers "F.Cu" "B.Cu")
+		(net "GND")
+	)
+	(via
+		(at 108.65 85.45)
+		(size 0.6)
+		(drill 0.3)
+		(layers "F.Cu" "B.Cu")
+		(free yes)
 		(net "GND")
 	)
@@
 		(layer "F.Cu")
 		(hatch edge 0.5)
-		(priority 4)
+		(priority 5)
 		(connect_pads yes
 			(clearance 0.2)
@@
 		(layer "F.Cu")
 		(hatch edge 0.5)
-		(priority 6)
+		(priority 7)
 		(connect_pads yes
 			(clearance 0.2)
@@
 		(layer "F.Cu")
 		(hatch edge 0.5)
-		(priority 5)
+		(priority 6)
 		(connect_pads yes
 			(clearance 0.2)
@@
 		(layer "F.Cu")
 		(hatch edge 0.5)
-		(priority 3)
+		(priority 4)
 		(connect_pads yes
 			(clearance 0.2)
@@
 		(layer "F.Cu")
 		(hatch edge 0.5)
-		(priority 2)
+		(priority 3)
 		(connect_pads yes
 			(clearance 0.2)
@@
 		(name "BuckIN")
 		(hatch edge 0.5)
-		(priority 1)
+		(priority 2)
 		(connect_pads yes
 			(clearance 0.2)
@@
 	)
 	(zone
-		(net "+3V3")
-		(layer "B.Cu")
+		(net "GND")
+		(layers "F.Cu" "B.Cu")
+		(name "GND_2")
 		(hatch edge 0.5)
-		(priority 7)
+		(connect_pads
+			(clearance 0.2)
+		)
+		(min_thickness 0.25)
+		(fill yes
+			(thermal_gap 0.3)
+			(thermal_bridge_width 0.3)
+			(island_removal_mode 0)
+		)
+		(polygon
+			(pts
+				(xy 152.85 80.25) (xy 152.85 120.05) (xy 86.45 120.05) (xy 86.45 80.25)
+			)
+		)
+	)
+	(zone
+		(net "+3V3")
+		(layer "B.Cu")
+		(hatch edge 0.5)
+		(priority 8)
 		(connect_pads yes
 			(clearance 0.2)
@@
 		(layer "B.Cu")
 		(hatch edge 0.5)
-		(priority 8)
+		(priority 9)
 		(connect_pads yes
 			(clearance 0.2)
@@
 		(net "GND")
 		(layers "In1.Cu" "In2.Cu")
-		(name "GND_2")
+		(name "GND_1")
 		(hatch edge 0.5)
+		(priority 1)
 		(connect_pads
 			(clearance 0.2)
